Commit message: 重命名 gz 仿真 ros2_control 宏，新增 description 显示 launch 文件
- load_gazebo_sim_ros2_control_plugin 宏更名为 gzbot_sim_ros2_control，同步更新 gzbot.urdf.xacro 引用
- 新增 gzbot_description.launch.py：robot_state_publisher + joint_state_publisher + RViz 显示

Co-Authored-By: Claude Code <noreply@anthropic.com>

File: src/gzbot_ros2/gzbot_description/urdf/control/gzbot_sim_ros2_control.urdf.xacro (robot description, xacro)
@@ -1,5 +1,5 @@
 <?xml version="1.0" ?>
 <robot xmlns:xacro="http://wiki.ros.org/xacro">
-    <xacro:macro name="load_gazebo_sim_ros2_control_plugin" params="use_gazebo">
+    <xacro:macro name="gzbot_sim_ros2_control" params="use_gazebo">
         <xacro:if value="${use_gazebo}">
             <gazebo>

File: src/gzbot_ros2/gzbot_description/urdf/robot/gzbot.urdf.xacro (robot description, xacro)
@@ -9,7 +9,6 @@
   <xacro:include filename="$(find gzbot_description)/urdf/control/gzbot_ros2_control.urdf.xacro" />
   <xacro:gzbot_ros2_control use_gazebo="$(arg use_gazebo)" />
-  <xacro:include
-    filename="$(find gzbot_description)/urdf/control/load_gazebo_sim_ros2_control_plugin.urdf.xacro" />
-  <xacro:load_gazebo_sim_ros2_control_plugin use_gazebo="$(arg use_gazebo)" />
+  <xacro:include filename="$(find gzbot_description)/urdf/control/gzbot_sim_ros2_control.urdf.xacro" />
+  <xacro:gzbot_sim_ros2_control use_gazebo="$(arg use_gazebo)" />
   <joint name="gripper_base_joint" type="fixed">
     <parent link="tool_link" />
