Commit message: 重构 URDF 目录 mesh→common/mech；修复夹爪控制并统一负值闭合
- ros2_controllers.yaml：gripper_controller 改为 position_controllers/GripperActionController（Humble 下 GripperCommand 的实际注册名），参数改为 joint 单值
- gzbot_gripper.urdf.xacro：右手指加回 URDF mimic 标签（供 robot_state_publisher 显示右手指）；左手指 axis 反向、限位 [-0.06, 0.0]，负值=闭合（与 mycobot 习惯一致），两侧 mimic 系数 +1.0
- gzbot_ros2_control.urdf.xacro：mimic multiplier 同步 +1.0
- mesh/ 三个 xacro 迁移至 mech/，新增 common/inertial_macros.urdf.xacro

Co-Authored-By: Claude Code <noreply@anthropic.com>

File: src/gzbot_ros2/gzbot_description/urdf/control/gzbot_ros2_control.urdf.xacro (robot description, xacro)
@@ -4,8 +4,8 @@
         <xacro:if value="${use_gazebo}">
             <ros2_control name="gzbot" type="system">
-                <hardware>
-                    <!-- By default, set up controllers for simulation. This won't work on real
-                    hardware -->
-                    <plugin>mock_components/GenericSystem</plugin>
+               <hardware>
+                    <xacro:if value="${use_gazebo}">
+                        <plugin>gz_ros2_control/GazeboSimSystem</plugin>
+                    </xacro:if>
                 </hardware>
                 <joint name="joint1">
@@ -50,4 +50,15 @@
                         <param name="initial_value">0.0</param>
                     </state_interface>
+                    <state_interface name="velocity" />
+                </joint>
+                <!-- 从动手指：cm 软件层 mimic，自动镜像左手指命令
+                     （gz 物理引擎会忽略 URDF 的 mimic 标签，联动靠这里） -->
+                <joint name="gripper_right_finger_joint">
+                    <param name="mimic">gripper_left_finger_joint</param>
+                    <param name="multiplier">1.0</param>
+                    <param name="offset">0.0</param>
+                    <command_interface name="position" />
+                    <state_interface name="position" />
+                    <state_interface name="velocity" />
                 </joint>
             </ros2_control>

File: src/gzbot_ros2/gzbot_description/urdf/mech/gzbot_arm.urdf.xacro (robot description, xacro)
@@ -4,4 +4,5 @@
         <!-- base_link: box size 0.4 0.4 0.1 -->
         <link name="base_link">
+            <xacro:box_inertial m="1.0" x="0.4" y="0.4" z="0.1" />
             <visual>
                 <geometry>
@@ -9,5 +10,7 @@
                 </geometry>
                 <origin xyz="0 0 0.05" rpy="0 0 0" />
-                <material name="grey" />
+                <material name="grey">
+                    <color rgba="0.5 0.5 0.5 1" />
+                </material>
             </visual>
             <collision>
@@ -18,9 +21,16 @@
             </collision>
         </link>
+        <!-- gz 材质写法（Gazebo/Orange 是 Gazebo Classic 专用，gz/ign 不识别） -->
         <gazebo reference="base_link">
-            <material>Gazebo/Orange</material>
+            <visual>
+                <material>
+                    <ambient>0.5 0.5 0.5 1</ambient>
+                    <diffuse>0.5 0.5 0.5 1</diffuse>
+                </material>
+            </visual>
         </gazebo>
         <!-- shoulder_link: cylinder length 0.5 radius 0.1 -->
         <link name="shoulder_link">
+            <xacro:cylinder_inertial m="0.5" r="0.1" l="0.5" />
             <visual>
                 <geometry>
@@ -28,5 +38,7 @@
                 </geometry>
                 <origin xyz="0 0 0.25" rpy="0 0 0" />
-                <material name="blue" />
+                <material name="blue">
+                    <color rgba="0 0 0.5 1" />
+                </material>
             </visual>
             <collision>
@@ -39,4 +51,5 @@
         <!-- arm_link: cylinder length 0.6 radius 0.05 -->
         <link name="arm_link">
+            <xacro:cylinder_inertial m="0.4" r="0.05" l="0.6" />
             <visual>
                 <geometry>
@@ -45,5 +58,7 @@
                 <!-- cylinder default along z, rotate to x direction -->
                 <origin xyz="0 0 0.3" rpy="0 0 0" />
-                <material name="grey" />
+                <material name="grey">
+                    <color rgba="0.5 0.5 0.5 1" />
+                </material>
             </visual>
             <collision>
@@ -56,4 +71,5 @@
         <!-- elbow_link: cylinder length 0.1 radius 0.05 -->
         <link name="elbow_link">
+            <xacro:cylinder_inertial m="0.1" r="0.05" l="0.1" />
             <visual>
                 <geometry>
@@ -61,5 +77,7 @@
                 </geometry>
                 <origin xyz="0 0 0.05" rpy="0 0 0" />
-                <material name="blue" />
+                <material name="blue">
+                    <color rgba="0 0 0.5 1" />
+                </material>
             </visual>
             <collision>
@@ -72,4 +90,5 @@
         <!-- forearm_link: cylinder length 0.5 radius 0.05 -->
         <link name="forearm_link">
+            <xacro:cylinder_inertial m="0.3" r="0.05" l="0.5" />
             <visual>
                 <geometry>
@@ -78,5 +97,7 @@
                 <!-- cylinder default along z, rotate to x direction -->
                 <origin xyz="0 0 0.25" rpy="0 0 0" />
-                <material name="grey" />
+                <material name="grey">
+                    <color rgba="0.5 0.5 0.5 1" />
+                </material>
             </visual>
             <collision>
@@ -89,4 +110,5 @@
         <!-- wrist_link: box size 0.1 0.1 0.05 -->
         <link name="wrist_link">
+            <xacro:box_inertial m="0.1" x="0.1" y="0.1" z="0.05" />
             <visual>
                 <geometry>
@@ -94,5 +116,7 @@
                 </geometry>
                 <origin xyz="0 0 0.025" rpy="0 0 0" />
-                <material name="blue" />
+                <material name="blue">
+                    <color rgba="0 0 0.5 1" />
+                </material>
             </visual>
             <collision>
@@ -105,4 +129,5 @@
         <!-- hand_link: box size 0.1 0.1 0.02 -->
         <link name="hand_link">
+            <xacro:box_inertial m="0.05" x="0.1" y="0.1" z="0.02" />
             <visual>
                 <geometry>
@@ -110,5 +135,7 @@
                 </geometry>
                 <origin xyz="0 0 0.01" rpy="0 0 0" />
-                <material name="grey" />
+                <material name="grey">
+                    <color rgba="0.5 0.5 0.5 1" />
+                </material>
             </visual>
             <collision>
@@ -119,6 +146,8 @@
             </collision>
         </link>
-        <!-- tool_link: no visual -->
-        <link name="tool_link" />
+        <!-- tool_link: no visual，占位惯性防零质量实体被拒 -->
+        <link name="tool_link">
+            <xacro:dummy_inertial />
+        </link>
         <!-- joint1: revolute, axis z, min -3.14, max 3.14 -->
         <joint name="joint1" type="revolute">

File: src/gzbot_ros2/gzbot_description/urdf/mech/gzbot_gripper.urdf.xacro (robot description, xacro)
@@ -4,4 +4,5 @@
         <!-- 夹爪底座 -->
         <link name="gripper_base_link">
+            <xacro:box_inertial m="0.1" x="0.20" y="0.06" z="0.02" />
             <visual>
                 <geometry>
@@ -9,5 +10,7 @@
                 </geometry>
                 <origin xyz="0 0 0.01" rpy="0 0 0" />
-                <material name="dark_green" />
+                <material name="dark_green">
+                    <color rgba="0 0.4 0 1" />
+                </material>
             </visual>
             <collision>
@@ -20,4 +23,5 @@
         <!-- 左夹爪手指 -->
         <link name="gripper_left_finger_link">
+            <xacro:box_inertial m="0.02" x="0.02" y="0.06" z="0.08" />
             <visual>
                 <geometry>
@@ -25,5 +29,7 @@
                 </geometry>
                 <origin xyz="0 0 0.04" rpy="0 0 0" />
-                <material name="light_green" />
+                <material name="light_green">
+                    <color rgba="0 0.6 0 1" />
+                </material>
             </visual>
             <collision>
@@ -36,4 +42,5 @@
         <!-- 右夹爪手指 -->
         <link name="gripper_right_finger_link">
+            <xacro:box_inertial m="0.02" x="0.02" y="0.06" z="0.08" />
             <visual>
                 <geometry>
@@ -41,5 +48,7 @@
                 </geometry>
                 <origin xyz="0 0 0.04" rpy="0 0 0" />
-                <material name="light_green" />
+                <material name="light_green">
+                    <color rgba="0 0.6 0 1" />
+                </material>
             </visual>
             <collision>
@@ -50,13 +59,14 @@
             </collision>
         </link>
-        <!-- 左手指连接到底座 -->
+        <!-- 左手指连接到底座（axis 朝外、零点=张开，负值=闭合，与 mycobot 习惯一致） -->
         <joint name="gripper_left_finger_joint" type="prismatic">
             <parent link="gripper_base_link" />
             <child link="gripper_left_finger_link" />
             <origin xyz="-0.07 0 0.02" rpy="0 0 0" />
-            <axis xyz="1 0 0" />
-            <limit effort="1000.0" velocity="1.0" lower="0.0" upper="0.06" />
+            <axis xyz="-1 0 0" />
+            <limit effort="1000.0" velocity="1.0" lower="-0.06" upper="0.0" />
         </joint>
-        <!-- 右手指连接到底座 -->
+        <!-- 右手指连接到底座（mimic 标签：gz 物理引擎会忽略，物理联动由 ros2_control 的 mimic param 实现；
+             此标签供 robot_state_publisher 显示右手指、MoveIt 解析用） -->
         <joint name="gripper_right_finger_joint" type="prismatic">
             <parent link="gripper_base_link" />
@@ -64,5 +74,5 @@
             <origin xyz="0.07 0 0.02" rpy="0 0 0" />
             <axis xyz="1 0 0" />
-            <mimic joint="gripper_left_finger_joint" multiplier="-1.0" />
+            <mimic joint="gripper_left_finger_joint" multiplier="1.0" offset="0.0" />
             <limit effort="1000.0" velocity="1.0" lower="-0.06" upper="0.0" />
         </joint>

File: src/gzbot_ros2/gzbot_description/urdf/robot/gzbot.urdf.xacro (robot description, xacro)
@@ -2,8 +2,9 @@
 <robot name="my_robot" xmlns:xacro="http://www.ros.org/wiki/xacro">
   <xacro:arg name="use_gazebo" default="false" />
-  <xacro:include filename="$(find gzbot_description)/urdf/mesh/common_properties.urdf.xacro" />
-  <xacro:include filename="$(find gzbot_description)/urdf/mesh/gzbot_arm.urdf.xacro" />
+  <xacro:include filename="$(find gzbot_description)/urdf/mech/common_properties.urdf.xacro" />
+  <xacro:include filename="$(find gzbot_description)/urdf/common/inertial_macros.urdf.xacro" />
+  <xacro:include filename="$(find gzbot_description)/urdf/mech/gzbot_arm.urdf.xacro" />
   <xacro:gzbot_arm />
-  <xacro:include filename="$(find gzbot_description)/urdf/mesh/gzbot_gripper.urdf.xacro" />
+  <xacro:include filename="$(find gzbot_description)/urdf/mech/gzbot_gripper.urdf.xacro" />
   <xacro:gzbot_gripper />
   <xacro:include filename="$(find gzbot_description)/urdf/control/gzbot_ros2_control.urdf.xacro" />
